File: STM32WB OpenThread test board/STM32WB OpenThread test board.kicad_pcb (KiCad board)
At the start: 2 copper layers, 15 parts, among them J1 Conn_Coaxial, U1 STM32WB55CC

Commit message: WIP
Parts:
- J1: footprint Connector_Coaxial:SMA_Amphenol_132203-12_Horizontal -> Connector_Coaxial:U.FL_Hirose_U.FL-R-SMT-1_Vertical
- moved J1 11.1 mm to (137.5, 114.8)
Other:
- board outline added: 40 x 30 mm
Changed lines of the file:
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@@
   (general
     (thickness 1.6)
-    (drawings 0)
+    (drawings 4)
     (tracks 0)
     (zones 0)
@@
     (add_net VDD)
   )
+  (module Connector_Coaxial:U.FL_Hirose_U.FL-R-SMT-1_Vertical (layer F.Cu)
+    (at 137.5 114.75 270)
+    (descr "Hirose U.FL Coaxial https://www.hirose.com/product/en/products/U.FL/U.FL-R-SMT-1%2810%29/")
+    (tags "Hirose U.FL Coaxial")
+    (attr smd)
+    (fp_text reference J1 (at 0.475 -3.2 90) (layer F.SilkS)
+      (effects (font (size 1 1) (thickness 0.15)))
+    )
+    (fp_text value Conn_Coaxial (at 0.475 3.2 90) (layer F.Fab)
+      (effects (font (size 1 1) (thickness 0.15)))
+    )
+    (fp_line (start -1.32 -1) (end -2.02 -1) (layer F.CrtYd) (width 0.05))
+    (fp_line (start -1.32 1.8) (end -1.32 1) (layer F.CrtYd) (width 0.05))
+    (fp_line (start -1.32 -1.8) (end -1.12 -1.8) (layer F.CrtYd) (width 0.05))
+    (fp_line (start -1.12 -1.8) (end -1.12 -2.5) (layer F.CrtYd) (width 0.05))
+    (fp_line (start 2.08 -2.5) (end -1.12 -2.5) (layer F.CrtYd) (width 0.05))
+    (fp_line (start -1.32 -1) (end -1.32 -1.8) (layer F.CrtYd) (width 0.05))
+    (fp_line (start 2.08 -1.8) (end 2.08 -2.5) (layer F.CrtYd) (width 0.05))
+    (fp_line (start 2.08 -1.8) (end 2.28 -1.8) (layer F.CrtYd) (width 0.05))
+    (fp_line (start -0.885 -1.4) (end -0.885 -0.76) (layer F.SilkS) (width 0.12))
+    (fp_line (start -0.425 1.5) (end -0.425 1.3) (layer F.Fab) (width 0.1))
+    (fp_line (start -0.425 1.3) (end -0.825 1.3) (layer F.Fab) (width 0.1))
+    (fp_line (start -0.825 0.3) (end -0.825 1.3) (layer F.Fab) (width 0.1))
+    (fp_line (start -1.075 0.3) (end -0.825 0.3) (layer F.Fab) (width 0.1))
+    (fp_line (start -1.075 0.3) (end -1.075 -0.15) (layer F.Fab) (width 0.1))
+    (fp_line (start -0.925 -0.3) (end -0.825 -0.3) (layer F.Fab) (width 0.1))
+    (fp_line (start -0.825 -0.3) (end -0.825 -1.3) (layer F.Fab) (width 0.1))
+    (fp_line (start -0.425 -1.5) (end -0.425 -1.3) (layer F.Fab) (width 0.1))
+    (fp_line (start -0.425 -1.3) (end -0.825 -1.3) (layer F.Fab) (width 0.1))
+    (fp_line (start -0.425 1.5) (end 1.375 1.5) (layer F.Fab) (width 0.1))
+    (fp_line (start 1.375 1.5) (end 1.375 1.3) (layer F.Fab) (width 0.1))
+    (fp_line (start 1.775 1.3) (end 1.375 1.3) (layer F.Fab) (width 0.1))
+    (fp_line (start 1.775 -1.3) (end 1.775 1.3) (layer F.Fab) (width 0.1))
+    (fp_line (start -0.425 -1.5) (end 1.375 -1.5) (layer F.Fab) (width 0.1))
+    (fp_line (start 1.375 -1.5) (end 1.375 -1.3) (layer F.Fab) (width 0.1))
+    (fp_line (start 1.775 -1.3) (end 1.375 -1.3) (layer F.Fab) (width 0.1))
+    (fp_line (start -0.925 -0.3) (end -1.075 -0.15) (layer F.Fab) (width 0.1))
+    (fp_line (start -0.885 1.4) (end -0.885 0.76) (layer F.SilkS) (width 0.12))
+    (fp_line (start -0.885 -0.76) (end -1.515 -0.76) (layer F.SilkS) (width 0.12))
+    (fp_line (start 1.835 -1.35) (end 1.835 1.35) (layer F.SilkS) (width 0.12))
+    (fp_line (start 2.08 2.5) (end -1.12 2.5) (layer F.CrtYd) (width 0.05))
+    (fp_line (start -1.12 2.5) (end -1.12 1.8) (layer F.CrtYd) (width 0.05))
+    (fp_line (start -1.32 1.8) (end -1.12 1.8) (layer F.CrtYd) (width 0.05))
+    (fp_line (start 2.28 1.8) (end 2.28 -1.8) (layer F.CrtYd) (width 0.05))
+    (fp_line (start 2.08 2.5) (end 2.08 1.8) (layer F.CrtYd) (width 0.05))
+    (fp_line (start 2.08 1.8) (end 2.28 1.8) (layer F.CrtYd) (width 0.05))
+    (fp_line (start -1.32 1) (end -2.02 1) (layer F.CrtYd) (width 0.05))
+    (fp_line (start -2.02 1) (end -2.02 -1) (layer F.CrtYd) (width 0.05))
+    (fp_text user %R (at 0.475 0) (layer F.Fab)
+      (effects (font (size 0.6 0.6) (thickness 0.09)))
+    )
+    (pad 2 smd rect (at 0.475 -1.475 270) (size 2.2 1.05) (layers F.Cu F.Paste F.Mask)
+      (net 2 GND))
+    (pad 1 smd rect (at -1.05 0 270) (size 1.05 1) (layers F.Cu F.Paste F.Mask)
+      (net 41 "Net-(J1-Pad1)"))
+    (pad 2 smd rect (at 0.475 1.475 270) (size 2.2 1.05) (layers F.Cu F.Paste F.Mask)
+      (net 2 GND))
+    (model ${KISYS3DMOD}/Connector_Coaxial.3dshapes/U.FL_Hirose_U.FL-R-SMT-1_Vertical.wrl
+      (offset (xyz 0.4749999928262157 0 0))
+      (scale (xyz 1 1 1))
+      (rotate (xyz 0 0 0))
+    )
+  )
   (module Package_DFN_QFN:QFN-48-1EP_7x7mm_P0.5mm_EP5.6x5.6mm (layer F.Cu)
     (at 134 104.25)
@@
     )
     (fp_text value STM32WB55CC (at 0 4.82) (layer F.Fab)
-      (effects (font (size 1 1) (thickness 0.15)))
-    )
-    (fp_text user %R (at 0 0) (layer F.Fab)
       (effects (font (size 1 1) (thickness 0.15)))
     )
@@
     (fp_line (start 4.12 4.12) (end 4.12 -4.12) (layer F.CrtYd) (width 0.05))
     (fp_line (start 4.12 -4.12) (end -4.12 -4.12) (layer F.CrtYd) (width 0.05))
+    (fp_text user %R (at 0 0) (layer F.Fab)
+      (effects (font (size 1 1) (thickness 0.15)))
+    )
     (pad "" smd roundrect (at 2.1 2.1) (size 1.13 1.13) (layers F.Paste) (roundrect_rratio 0.221239))
     (pad "" smd roundrect (at 2.1 0.7) (size 1.13 1.13) (layers F.Paste) (roundrect_rratio 0.221239))
@@
     )
   )
-  (module Connector_Coaxial:SMA_Amphenol_132203-12_Horizontal (layer F.Cu)
-    (at 137.0965 125.7935 270)
-    (descr https://www.amphenolrf.com/media/downloads/1769/132203-12.pdf)
-    (tags "SMA THT Female Jack Horizontal")
-    (fp_text reference J1 (at -5.2 0) (layer F.SilkS)
-      (effects (font (size 1 1) (thickness 0.15)))
-    )
-    (fp_text value Conn_Coaxial (at 0 5 90) (layer F.Fab)
-      (effects (font (size 1 1) (thickness 0.15)))
-    )
-    (fp_line (start -3.175 -5.998) (end 3.175 -6.704) (layer F.Fab) (width 0.1))
-    (fp_line (start -3.175 -6.704) (end 3.175 -7.41) (layer F.Fab) (width 0.1))
-    (fp_line (start -3.175 -7.41) (end 3.175 -8.116) (layer F.Fab) (width 0.1))
-    (fp_line (start -3.175 -8.116) (end 3.175 -8.822) (layer F.Fab) (width 0.1))
-    (fp_line (start -3.175 -8.822) (end 3.175 -9.528) (layer F.Fab) (width 0.1))
-    (fp_line (start -3.175 -9.528) (end 3.175 -10.234) (layer F.Fab) (width 0.1))
-    (fp_line (start -3.175 -10.234) (end 3.175 -10.94) (layer F.Fab) (width 0.1))
-    (fp_line (start -3.175 -10.94) (end 3.175 -11.646) (layer F.Fab) (width 0.1))
-    (fp_line (start -3.175 -11.646) (end 3.175 -12.352) (layer F.Fab) (width 0.1))
-    (fp_line (start -3.175 -12.352) (end 3.175 -13.058) (layer F.Fab) (width 0.1))
-    (fp_line (start -3.175 -13.058) (end 3.175 -13.764) (layer F.Fab) (width 0.1))
-    (fp_line (start -3.175 -13.764) (end 3.175 -14.47) (layer F.Fab) (width 0.1))
-    (fp_line (start -3.175 -14.47) (end 3.175 -15.176) (layer F.Fab) (width 0.1))
-    (fp_line (start -3.175 -15.176) (end 3.175 -15.882) (layer F.Fab) (width 0.1))
-    (fp_line (start -3.175 -15.882) (end 3.175 -16.588) (layer F.Fab) (width 0.1))
-    (fp_line (start -3.175 -16.588) (end 3.175 -17.294) (layer F.Fab) (width 0.1))
-    (fp_line (start -3.175 -17.294) (end 3.175 -18) (layer F.Fab) (width 0.1))
-    (fp_line (start 4.5 4.5) (end -4.5 4.5) (layer F.CrtYd) (width 0.05))
-    (fp_line (start 4.5 4.5) (end 4.5 -20) (layer F.CrtYd) (width 0.05))
-    (fp_line (start -4.5 -20) (end -4.5 4.5) (layer F.CrtYd) (width 0.05))
-    (fp_line (start -4.5 -20) (end 4.5 -20) (layer F.CrtYd) (width 0.05))
-    (fp_line (start -4 -4) (end -4 4) (layer F.Fab) (width 0.1))
-    (fp_line (start -4 4) (end 4 4) (layer F.Fab) (width 0.1))
-    (fp_line (start 4 -4) (end 4 4) (layer F.Fab) (width 0.1))
-    (fp_line (start -4.15 -4.15) (end -4.15 4.15) (layer F.SilkS) (width 0.12))
-    (fp_line (start 4.15 -4.15) (end 4.15 4.15) (layer F.SilkS) (width 0.12))
-    (fp_line (start -4.15 4.15) (end 4.15 4.15) (layer F.SilkS) (width 0.12))
-    (fp_line (start -4.15 -4.15) (end 4.15 -4.15) (layer F.SilkS) (width 0.12))
-    (fp_line (start -3.175 -19.5) (end 3.175 -19.5) (layer F.Fab) (width 0.1))
-    (fp_line (start -3.175 -19.5) (end -3.175 -5.07) (layer F.Fab) (width 0.1))
-    (fp_line (start 3.175 -19.5) (end 3.175 -5.07) (layer F.Fab) (width 0.1))
-    (fp_line (start 3.9 -4) (end 3.9 -5.07) (layer F.Fab) (width 0.1))
-    (fp_line (start 3.9 -5.07) (end -3.9 -5.07) (layer F.Fab) (width 0.1))
-    (fp_line (start -3.9 -5.07) (end -3.9 -4) (layer F.Fab) (width 0.1))
-    (fp_line (start -4 -4) (end 4 -4) (layer F.Fab) (width 0.1))
-    (fp_line (start -3.175 -18) (end 3.175 -18.706) (layer F.Fab) (width 0.1))
-    (fp_text user %R (at 0 0 90) (layer F.Fab)
-      (effects (font (size 1 1) (thickness 0.15)))
-    )
-    (pad 1 thru_hole circle (at 0 0 270) (size 2.25 2.25) (drill 1.5) (layers *.Cu *.Mask)
-      (net 41 "Net-(J1-Pad1)"))
-    (pad 2 thru_hole circle (at 2.54 2.54) (size 2.25 2.25) (drill 1.7) (layers *.Cu *.Mask)
-      (net 2 GND))
-    (pad 2 thru_hole circle (at 2.54 -2.54 270) (size 2.25 2.25) (drill 1.7) (layers *.Cu *.Mask)
-      (net 2 GND))
-    (pad 2 thru_hole circle (at -2.54 -2.54 270) (size 2.25 2.25) (drill 1.7) (layers *.Cu *.Mask)
-      (net 2 GND))
-    (pad 2 thru_hole circle (at -2.54 2.54 270) (size 2.25 2.25) (drill 1.7) (layers *.Cu *.Mask)
-      (net 2 GND))
-    (model ${KISYS3DMOD}/Connector_Coaxial.3dshapes/SMA_Amphenol_132203-12_Horizontal.wrl
-      (at (xyz 0 0 0))
-      (scale (xyz 1 1 1))
-      (rotate (xyz 0 0 0))
-    )
-  )
   (module Resistor_SMD:R_0402_1005Metric_Pad0.72x0.64mm_HandSolder (layer F.Cu)
     (at 143.3395 102.5845)
@@
     )
   )
+  (gr_line (start 160 90) (end 160 120) (layer Edge.Cuts) (width 0.1))
+  (gr_line (start 120 90) (end 160 90) (layer Edge.Cuts) (width 0.1))
+  (gr_line (start 120 120) (end 120 90) (layer Edge.Cuts) (width 0.1))
+  (gr_line (start 160 120) (end 120 120) (layer Edge.Cuts) (width 0.1))
 )
